Commit message: Version 1.1

File: franka_description/robots/franka_panda_fem_simple_v4_with_arm.urdf (robot description, URDF)
Before this commit: robot panda, 17 links, 16 joints
Joints:
- joint panda_left_finger_joint: limit lower=0.0 upper=0.04 effort=1e9 velocity=1e9 -> lower=-0.005 upper=0.04 effort=1e9 velocity=1e9
- joint panda_right_finger_joint: limit lower=0.0 upper=0.04 effort=1e9 velocity=1e9 -> lower=-0.005 upper=0.04 effort=1e9 velocity=1e9
